Commit message: clean urdf tree with manully measured sizes and add some fixmes

File: leap_hand_description/robots/leap_hand_left.xacro (robot description, xacro)
@@ -5,17 +5,23 @@
       <joint name="${prefix}_joint_${connected_to}" type="fixed">
         <parent link="${connected_to}"/>
-        <child link="${prefix}_base"/>
+        <child link="${prefix}_mount"/>
         <origin rpy="${rpy}" xyz="${xyz}"/>
       </joint>
     </xacro:unless>
+    <link name="${prefix}_mount"/>
+    <joint name="${prefix}_mount_joint" type="fixed">
+      <parent link="${prefix}_mount"/>
+      <child link="${prefix}_base"/>
+      <origin xyz="0.023 0.005 -0.038" rpy="0 0 0"/>
+    </joint>
     <link name="${prefix}_base"/>
     <joint name="${prefix}_base_joint" type="fixed">
       <parent link="${prefix}_base"/>
       <child link="${prefix}_palm_lower"/>
-      <origin xyz="0.015 0.055 0.17" rpy="0 -1.57079 0"/>
+      <origin xyz="0.0 0.0 0.04" rpy="0 0 0"/>
     </joint>
     <link name="${prefix}_palm_lower">
       <visual>
-        <origin xyz="-0.0955 -0.1170 0.0207" rpy="1.57079 0 3.14159" />
+        <origin rpy="1.17365 1.57079 2.74446" xyz="-0.00570 -0.06200 0.03450"/>
         <geometry>
           <mesh filename="package://${description_pkg}/meshes/visual/palm_lower_left.obj"/>
@@ -23,5 +29,5 @@
       </visual>
       <collision>
-        <origin xyz="-0.0848 -0.0996 0.0152" rpy="0 0 0"/>
+        <origin rpy="0.00000 -1.57079 0.00000" xyz="-0.00020 -0.04460 0.04520"/>
         <geometry>
           <box size="0.022 0.026 0.034"/>
@@ -29,5 +35,5 @@
       </collision>
       <collision>
-        <origin xyz="-0.0848 -0.0546 0.0152" rpy="0 0 0"/>
+        <origin rpy="0.00000 -1.57079 0.00000" xyz="-0.00020 0.00040 0.04520"/>
         <geometry>
           <box size="0.022 0.026 0.034"/>
@@ -35,5 +41,5 @@
       </collision>
       <collision>
-        <origin xyz="-0.0848 -0.0096 0.0152" rpy="0 0 0"/>
+        <origin rpy="0.00000 -1.57079 0.00000" xyz="-0.00020 0.04540 0.04520"/>
         <geometry>
           <box size="0.022 0.026 0.034"/>
@@ -41,5 +47,5 @@
       </collision>
       <collision>
-        <origin xyz="-0.1428 -0.0126 0.0147" rpy="0 0 0.2967"/>
+        <origin rpy="-1.57077 -1.27410 1.57078" xyz="0.00030 0.04240 -0.01280"/>
         <geometry>
           <box size="0.058 0.02 0.046"/>
@@ -47,5 +53,5 @@
       </collision>
       <collision>
-        <origin xyz="-0.1058 -0.0555 0.0232" rpy="0 0 0"/>
+        <origin rpy="0.00000 -1.57079 0.00000" xyz="-0.00820 -0.00050 0.02420"/>
         <geometry>
           <box size="0.02 0.12 0.03"/>
@@ -53,5 +59,5 @@
       </collision>
       <collision>
-        <origin xyz="-0.1078 -0.0555 0.0002" rpy="0 0.785 0"/>
+        <origin rpy="0.00000 -0.78579 0.00000" xyz="0.01480 -0.00050 0.02220"/>
         <geometry>
           <box size="0.01 0.12 0.02"/>
@@ -59,5 +65,5 @@
       </collision>
       <collision>
-        <origin xyz="-0.1238 -0.0575 0.0147" rpy="0 0 0"/>
+        <origin rpy="0.00000 -1.57079 0.00000" xyz="0.00030 -0.00250 0.00620"/>
         <geometry>
           <box size="0.024 0.116 0.046"/>
@@ -65,5 +71,5 @@
       </collision>
       <collision>
-        <origin xyz="-0.1538 -0.0375 0.0147" rpy="0 0 0"/>
+        <origin rpy="0.00000 -1.57079 0.00000" xyz="0.00030 0.01750 -0.02380"/>
         <geometry>
           <box size="0.044 0.052 0.046"/>
@@ -71,5 +77,5 @@
       </collision>
       <collision>
-        <origin xyz="-0.1738 -0.0815 0.0202" rpy="0 0 0"/>
+        <origin rpy="0.00000 -1.57079 0.00000" xyz="-0.00520 -0.02650 -0.04380"/>
         <geometry>
           <box size="0.004 0.036 0.034"/>
@@ -77,5 +83,5 @@
       </collision>
       <collision>
-        <origin xyz="-0.1538 -0.0875 0.0362" rpy="0 0 0"/>
+        <origin rpy="0.00000 -1.57079 0.00000" xyz="-0.02120 -0.03250 -0.02380"/>
         <geometry>
           <box size="0.044 0.056 0.004"/>
@@ -83,5 +89,5 @@
       </collision>
       <inertial>
-        <origin xyz="0 0 0" rpy="0 0 0"/>
+        <origin rpy="0.00000 -1.57079 0.00000" xyz="0.01500 0.05500 0.13000"/>
         <mass value="0.235"/>
         <inertia ixx="0.000351007" ixy="-0.000001393" ixz="-0.000000694" iyy="0.000523205" iyz="-0.000003085" izz="0.000256996"/>
@@ -245,6 +251,6 @@
     </joint>
     <joint name="${prefix}_1" type="revolute">
-      <origin xyz="-0.0825 -0.0857 0.0078" rpy="1.57079 1.57079 0"/>
-      <parent link="${prefix}_palm_lower"/>
+      <origin rpy="1.57079 0.00000 0.00000" xyz="0.00720 -0.03070 0.08750"/>
+      <parent link="${prefix}_base"/>
       <child link="${prefix}_mcp_joint"/>
       <axis xyz="0 0 -1"/>
@@ -425,6 +431,6 @@
     </joint>
     <joint name="${prefix}_5" type="revolute">
-      <origin xyz="-0.0825 -0.0403 0.0078" rpy="1.57079 1.57079 0"/>
-      <parent link="${prefix}_palm_lower"/>
+      <origin rpy="1.57079 0.00000 0.00000" xyz="0.00720 0.01470 0.08750"/>
+      <parent link="${prefix}_base"/>
       <child link="${prefix}_mcp_joint_2"/>
       <axis xyz="0 0 -1"/>
@@ -605,6 +611,6 @@
     </joint>
     <joint name="${prefix}_9" type="revolute">
-      <origin xyz="-0.0825 0.0051 0.0078" rpy="1.57079 1.57079 0"/>
-      <parent link="${prefix}_palm_lower"/>
+      <origin rpy="1.57079 0.00000 0.00000" xyz="0.00720 0.06010 0.08750"/>
+      <parent link="${prefix}_base"/>
       <child link="${prefix}_mcp_joint_3"/>
       <axis xyz="0 0 -1"/>
@@ -759,6 +765,6 @@
     </link>
     <joint name="${prefix}_12" type="revolute">
-      <origin xyz="-0.1448 -0.0900 0.0049" rpy="0 1.57079 0"/>
-      <parent link="${prefix}_palm_lower"/>
+      <origin rpy="0.00000 0.00000 0.00000" xyz="0.01010 -0.03500 0.02520"/>
+      <parent link="${prefix}_base"/>
       <child link="${prefix}_thumb_temp_base"/>
       <axis xyz="0 0 -1"/>

File: leap_hand_description/robots/leap_hand_right.xacro (robot description, xacro)
@@ -5,17 +5,23 @@
       <joint name="${prefix}_joint_${connected_to}" type="fixed">
         <parent link="${connected_to}"/>
-        <child link="${prefix}_base"/>
+        <child link="${prefix}_mount"/>
         <origin rpy="${rpy}" xyz="${xyz}"/>
       </joint>
     </xacro:unless>
+    <link name="${prefix}_mount"/>
+    <joint name="${prefix}_mount_joint" type="fixed">
+      <parent link="${prefix}_mount"/>
+      <child link="${prefix}_base"/>
+      <origin xyz="0.023 -0.005 -0.038" rpy="0 0 0"/>
+    </joint>
     <link name="${prefix}_base"/>
     <joint name="${prefix}_base_joint" type="fixed">
       <parent link="${prefix}_base"/>
       <child link="${prefix}_palm_lower"/>
-      <origin xyz="0 0.038 0.098" rpy="0 -1.57079 0"/>
+      <origin xyz="0.0 0.0 0.04" rpy="0 0 0"/>
     </joint>
     <link name="${prefix}_palm_lower">
       <visual>
-        <origin xyz="-0.0200 0.02575 -0.0347" rpy="0 0 0"/>
+        <origin rpy="0.00000 -1.57079 0.00000" xyz="0.02370 0.06375 0.03800"/>
         <geometry>
           <mesh filename="package://${description_pkg}/meshes/visual/palm_lower.obj"/>
@@ -23,5 +29,5 @@
       </visual>
       <collision>     <!-- palm_lower -->
-        <origin xyz="-0.009 0.008 -0.011" rpy="0 0 0"/>
+        <origin rpy="0.00000 -1.57079 0.00000" xyz="-0.00000 0.04600 0.04900"/>
         <geometry>
           <box size="0.022 0.026 0.034"/>
@@ -29,5 +35,6 @@
       </collision>
       <collision>
-        <origin xyz="-0.009 -0.037 -0.011" rpy="0 0 0"/>
+        <!-- <origin xyz="-0.009 -0.037 -0.011" rpy="0 0 0"/> -->
+        <origin rpy="0.00000 -1.57079 0.00000" xyz="-0.00000 0.00100 0.04900"/>
         <geometry>
           <box size="0.022 0.026 0.034"/>
@@ -35,5 +42,6 @@
       </collision>
       <collision>
-        <origin xyz="-0.009 -0.082 -0.011" rpy="0 0 0"/>
+        <!-- <origin xyz="-0.009 -0.082 -0.011" rpy="0 0 0"/> -->
+        <origin rpy="0.00000 -1.57079 0.00000" xyz="-0.00000 -0.04400 0.04900"/>
         <geometry>
           <box size="0.022 0.026 0.034"/>
@@ -41,5 +49,6 @@
       </collision>
       <collision>
-        <origin xyz="-0.066 -0.078 -0.0115" rpy="0 0 -0.2967"/>
+        <!-- <origin xyz="-0.066 -0.078 -0.0115" rpy="0 0 -0.2967"/> -->
+        <origin rpy="1.57077 -1.27410 -1.57078" xyz="0.00050 -0.04000 -0.00800"/>
         <geometry>
           <box size="0.058 0.02 0.046"/>
@@ -47,5 +56,6 @@
       </collision>
       <collision>
-        <origin xyz="-0.03 -0.035 -0.003" rpy="0 0 0"/>
+        <!-- <origin xyz="-0.03 -0.035 -0.003" rpy="0 0 0"/> -->
+        <origin rpy="0.00000 -1.57079 0.00000" xyz="-0.00800 0.00300 0.02800"/>
         <geometry>
           <box size="0.02 0.12 0.03"/>
@@ -53,5 +63,6 @@
       </collision>
       <collision>
-        <origin xyz="-0.032 -0.035 -0.024" rpy="0 0.785 0"/>
+        <!-- <origin xyz="-0.032 -0.035 -0.024" rpy="0 0.785 0"/> -->
+        <origin rpy="0.00000 -0.78579 0.00000" xyz="0.01300 0.00300 0.02600"/>
         <geometry>
           <box size="0.01 0.12 0.02"/>
@@ -59,5 +70,6 @@
       </collision>
       <collision>
-        <origin xyz="-0.048 -0.033 -0.0115" rpy="0 0 0"/>
+        <!-- <origin xyz="-0.048 -0.033 -0.0115" rpy="0 0 0"/> -->
+        <origin rpy="0.00000 -1.57079 0.00000" xyz="0.00050 0.00500 0.01000"/>
         <geometry>
           <box size="0.024 0.116 0.046"/>
@@ -65,5 +77,6 @@
       </collision>
       <collision>
-        <origin xyz="-0.078 -0.053 -0.0115" rpy="0 0 0"/>
+        <!-- <origin xyz="-0.078 -0.053 -0.0115" rpy="0 0 0"/> -->
+        <origin rpy="0.00000 -1.57079 0.00000" xyz="0.00050 -0.01500 -0.02000"/>
         <geometry>
           <box size="0.044 0.052 0.046"/>
@@ -71,5 +84,6 @@
       </collision>
       <collision>
-        <origin xyz="-0.098 -0.009 -0.006" rpy="0 0 0"/>
+        <!-- <origin xyz="-0.098 -0.009 -0.006" rpy="0 0 0"/> -->
+        <origin rpy="0.00000 -1.57079 0.00000" xyz="-0.00500 0.02900 -0.04000"/>
         <geometry>
           <box size="0.004 0.036 0.034"/>
@@ -77,5 +91,6 @@
       </collision>
       <collision>
-        <origin xyz="-0.078 -0.003 0.01" rpy="0 0 0"/>
+        <!-- <origin xyz="-0.078 -0.003 0.01" rpy="0 0 0"/> -->
+        <origin rpy="0.00000 -1.57079 0.00000" xyz="-0.02100 0.03500 -0.02000"/>
         <geometry>
           <box size="0.044 0.056 0.004"/>
@@ -83,5 +98,6 @@
       </collision>
       <inertial>
-        <origin xyz="0 0 0" rpy="0 0 0"/>
+        <!-- <origin xyz="0 0 0" rpy="0 0 0"/> -->
+        <origin rpy="0.00000 -1.57079 0.00000" xyz="-0.01100 0.03800 0.05800"/>
         <mass value="0.237"/>
         <inertia ixx="0.000354094" ixy="-0.000001193" ixz="-0.000002445" iyy="0.000260915" iyz="-0.000002905" izz="0.000529257"/>
@@ -245,6 +261,6 @@
     </joint>
     <joint name="${prefix}_1" type="revolute">
-      <origin xyz="-0.0070 0.0230 -0.0187" rpy="1.57079 1.57079 0"/>
-      <parent link="${prefix}_palm_lower"/>
+      <origin rpy="1.57079 0.00000 0.00000" xyz="0.00770 0.06100 0.09100"/>
+      <parent link="${prefix}_base"/>
       <child link="${prefix}_mcp_joint"/>
       <axis xyz="0 0 -1"/>
@@ -425,6 +441,6 @@
     </joint>
     <joint name="${prefix}_5" type="revolute">
-      <origin xyz="-0.0071 -0.0224 -0.0187" rpy="1.57079 1.57079 0"/>
-      <parent link="${prefix}_palm_lower"/>
+      <origin rpy="1.57079 0.00000 0.00000" xyz="0.00770 0.01560 0.09090"/>
+      <parent link="${prefix}_base"/>
       <child link="${prefix}_mcp_joint_2"/>
       <axis xyz="0 0 -1"/>
@@ -605,6 +621,6 @@
     </joint>
     <joint name="${prefix}_9" type="revolute">
-      <origin xyz="-0.00709 -0.0678 -0.0187" rpy="1.57079 1.57079 0"/>
-      <parent link="${prefix}_palm_lower"/>
+      <origin rpy="1.57079 0.00000 0.00000" xyz="0.00770 -0.02980 0.09091"/>
+      <parent link="${prefix}_base"/>
       <child link="${prefix}_mcp_joint_3"/>
       <axis xyz="0 0 -1"/>
@@ -759,6 +775,6 @@
     </link>
     <joint name="${prefix}_12" type="revolute">
-      <origin xyz="-0.0693 -0.0012 -0.0216" rpy="0 1.57079 0"/>
-      <parent link="${prefix}_palm_lower"/>
+      <origin rpy="0.00000 0.00000 0.00000" xyz="0.01060 0.03680 0.02870"/>
+      <parent link="${prefix}_base"/>
       <child link="${prefix}_thumb_temp_base"/>
       <axis xyz="0 0 -1"/>

Commit message: fix minor bugs and rename palm links in xacro; format launch

File: leap_hand_description/robots/leap_hand_left.xacro (robot description, xacro)
@@ -18,8 +18,8 @@
     <joint name="${prefix}_base_joint" type="fixed">
       <parent link="${prefix}_base"/>
-      <child link="${prefix}_palm_lower"/>
+      <child link="${prefix}_palm"/>
       <origin xyz="0.0 0.0 0.04" rpy="0 0 0"/>
     </joint>
-    <link name="${prefix}_palm_lower">
+    <link name="${prefix}_palm">
       <visual>
         <origin rpy="1.17365 1.57079 2.74446" xyz="-0.00570 -0.06200 0.03450"/>
@@ -248,5 +248,5 @@
       <axis xyz="0 0 -1"/>
       <limit effort="0.95" velocity="8.48" lower="-1.047" upper="1.047"/>
-      <joint_properties friction="0.0"/>
+      <dynamics friction="0.0"/>
     </joint>
     <joint name="${prefix}_1" type="revolute">
@@ -256,5 +256,5 @@
       <axis xyz="0 0 -1"/>
       <limit effort="0.95" velocity="8.48" lower="-0.314" upper="2.23"/>
-      <joint_properties friction="0.0"/>
+      <dynamics friction="0.0"/>
     </joint>
     <joint name="${prefix}_2" type="revolute">
@@ -264,5 +264,5 @@
       <axis xyz="0 0 -1"/>
       <limit effort="0.95" velocity="8.48" lower="-0.506" upper="1.885"/>
-      <joint_properties friction="0.0"/>
+      <dynamics friction="0.0"/>
     </joint>
     <joint name="${prefix}_3" type="revolute">
@@ -272,5 +272,5 @@
       <axis xyz="0 0 -1"/>
       <limit effort="0.95" velocity="8.48" lower="-0.366" upper="2.042"/>
-      <joint_properties friction="0.0"/>
+      <dynamics friction="0.0"/>
     </joint>
     <link name="${prefix}_mcp_joint_2">
@@ -428,5 +428,5 @@
       <axis xyz="0 0 -1"/>
       <limit effort="0.95" velocity="8.48" lower="-1.047" upper="1.047"/>
-      <joint_properties friction="0.0"/>
+      <dynamics friction="0.0"/>
     </joint>
     <joint name="${prefix}_5" type="revolute">
@@ -436,5 +436,5 @@
       <axis xyz="0 0 -1"/>
       <limit effort="0.95" velocity="8.48" lower="-0.314" upper="2.23"/>
-      <joint_properties friction="0.0"/>
+      <dynamics friction="0.0"/>
     </joint>
     <joint name="${prefix}_6" type="revolute">
@@ -444,5 +444,5 @@
       <axis xyz="0 0 -1"/>
       <limit effort="0.95" velocity="8.48" lower="-0.506" upper="1.885"/>
-      <joint_properties friction="0.0"/>
+      <dynamics friction="0.0"/>
     </joint>
     <joint name="${prefix}_7" type="revolute">
@@ -452,5 +452,5 @@
       <axis xyz="0 0 -1"/>
       <limit effort="0.95" velocity="8.48" lower="-0.366" upper="2.042"/>
-      <joint_properties friction="0.0"/>
+      <dynamics friction="0.0"/>
     </joint>
     <link name="${prefix}_mcp_joint_3">
@@ -608,5 +608,5 @@
       <axis xyz="0 0 -1"/>
       <limit effort="0.95" velocity="8.48" lower="-1.047" upper="1.047"/>
-      <joint_properties friction="0.0"/>
+      <dynamics friction="0.0"/>
     </joint>
     <joint name="${prefix}_9" type="revolute">
@@ -616,5 +616,5 @@
       <axis xyz="0 0 -1"/>
       <limit effort="0.95" velocity="8.48" lower="-0.314" upper="2.23"/>
-      <joint_properties friction="0.0"/>
+      <dynamics friction="0.0"/>
     </joint>
     <joint name="${prefix}_10" type="revolute">
@@ -624,5 +624,5 @@
       <axis xyz="0 0 -1"/>
       <limit effort="0.95" velocity="8.48" lower="-0.506" upper="1.885"/>
-      <joint_properties friction="0.0"/>
+      <dynamics friction="0.0"/>
     </joint>
     <joint name="${prefix}_11" type="revolute">
@@ -632,5 +632,5 @@
       <axis xyz="0 0 -1"/>
       <limit effort="0.95" velocity="8.48" lower="-0.366" upper="2.042"/>
-      <joint_properties friction="0.0"/>
+      <dynamics friction="0.0"/>
     </joint>
     <link name="${prefix}_thumb_temp_base">
@@ -770,5 +770,5 @@
       <axis xyz="0 0 -1"/>
       <limit effort="0.95" velocity="8.48" lower="-2.094" upper="0.349"/>
-      <joint_properties friction="0.0"/>
+      <dynamics friction="0.0"/>
     </joint>
     <joint name="${prefix}_13" type="revolute">
@@ -778,5 +778,5 @@
       <axis xyz="0 0 -1"/>
       <limit effort="0.95" velocity="8.48" lower="-2.443" upper="0.47"/>
-      <joint_properties friction="0.0"/>
+      <dynamics friction="0.0"/>
     </joint>
     <joint name="${prefix}_14" type="revolute">
@@ -786,5 +786,5 @@
       <axis xyz="0 0 -1"/>
       <limit effort="0.95" velocity="8.48" lower="-1.20" upper="1.90"/>
-      <joint_properties friction="0.0"/>
+      <dynamics friction="0.0"/>
     </joint>
     <joint name="${prefix}_15" type="revolute">
@@ -794,5 +794,5 @@
       <axis xyz="0 0 -1"/>
       <limit effort="0.95" velocity="8.48" lower="-1.34" upper="1.88"/>
-      <joint_properties friction="0.0"/>
+      <dynamics friction="0.0"/>
     </joint>
     <!--  virtual auxiliary link-->

File: leap_hand_description/robots/leap_hand_right.xacro (robot description, xacro)
@@ -18,8 +18,8 @@
     <joint name="${prefix}_base_joint" type="fixed">
       <parent link="${prefix}_base"/>
-      <child link="${prefix}_palm_lower"/>
+      <child link="${prefix}_palm"/>
       <origin xyz="0.0 0.0 0.04" rpy="0 0 0"/>
     </joint>
-    <link name="${prefix}_palm_lower">
+    <link name="${prefix}_palm">
       <visual>
         <origin rpy="0.00000 -1.57079 0.00000" xyz="0.02370 0.06375 0.03800"/>
@@ -28,5 +28,5 @@
         </geometry>
       </visual>
-      <collision>     <!-- palm_lower -->
+      <collision>
         <origin rpy="0.00000 -1.57079 0.00000" xyz="-0.00000 0.04600 0.04900"/>
         <geometry>
@@ -258,5 +258,5 @@
       <axis xyz="0 0 -1"/>
       <limit effort="0.95" velocity="8.48" lower="-1.047" upper="1.047"/>
-      <joint_properties friction="0.0"/>
+      <dynamics friction="0.0"/>
     </joint>
     <joint name="${prefix}_1" type="revolute">
@@ -266,5 +266,5 @@
       <axis xyz="0 0 -1"/>
       <limit effort="0.95" velocity="8.48" lower="-0.314" upper="2.23"/>
-      <joint_properties friction="0.0"/>
+      <dynamics friction="0.0"/>
     </joint>
     <joint name="${prefix}_2" type="revolute">
@@ -274,5 +274,5 @@
       <axis xyz="0 0 -1"/>
       <limit effort="0.95" velocity="8.48" lower="-0.506" upper="1.885"/>
-      <joint_properties friction="0.0"/>
+      <dynamics friction="0.0"/>
     </joint>
     <joint name="${prefix}_3" type="revolute">
@@ -282,5 +282,5 @@
       <axis xyz="0 0 -1"/>
       <limit effort="0.95" velocity="8.48" lower="-0.366" upper="2.042"/>
-      <joint_properties friction="0.0"/>
+      <dynamics friction="0.0"/>
     </joint>
     <link name="${prefix}_mcp_joint_2">
@@ -438,5 +438,5 @@
       <axis xyz="0 0 -1"/>
       <limit effort="0.95" velocity="8.48" lower="-1.047" upper="1.047"/>
-      <joint_properties friction="0.0"/>
+      <dynamics friction="0.0"/>
     </joint>
     <joint name="${prefix}_5" type="revolute">
@@ -446,5 +446,5 @@
       <axis xyz="0 0 -1"/>
       <limit effort="0.95" velocity="8.48" lower="-0.314" upper="2.23"/>
-      <joint_properties friction="0.0"/>
+      <dynamics friction="0.0"/>
     </joint>
     <joint name="${prefix}_6" type="revolute">
@@ -454,5 +454,5 @@
       <axis xyz="0 0 -1"/>
       <limit effort="0.95" velocity="8.48" lower="-0.506" upper="1.885"/>
-      <joint_properties friction="0.0"/>
+      <dynamics friction="0.0"/>
     </joint>
     <joint name="${prefix}_7" type="revolute">
@@ -462,5 +462,5 @@
       <axis xyz="0 0 -1"/>
       <limit effort="0.95" velocity="8.48" lower="-0.366" upper="2.042"/>
-      <joint_properties friction="0.0"/>
+      <dynamics friction="0.0"/>
     </joint>
     <link name="${prefix}_mcp_joint_3">
@@ -618,5 +618,5 @@
       <axis xyz="0 0 -1"/>
       <limit effort="0.95" velocity="8.48" lower="-1.047" upper="1.047"/>
-      <joint_properties friction="0.0"/>
+      <dynamics friction="0.0"/>
     </joint>
     <joint name="${prefix}_9" type="revolute">
@@ -626,5 +626,5 @@
       <axis xyz="0 0 -1"/>
       <limit effort="0.95" velocity="8.48" lower="-0.314" upper="2.23"/>
-      <joint_properties friction="0.0"/>
+      <dynamics friction="0.0"/>
     </joint>
     <joint name="${prefix}_10" type="revolute">
@@ -634,5 +634,5 @@
       <axis xyz="0 0 -1"/>
       <limit effort="0.95" velocity="8.48" lower="-0.506" upper="1.885"/>
-      <joint_properties friction="0.0"/>
+      <dynamics friction="0.0"/>
     </joint>
     <joint name="${prefix}_11" type="revolute">
@@ -642,5 +642,5 @@
       <axis xyz="0 0 -1"/>
       <limit effort="0.95" velocity="8.48" lower="-0.366" upper="2.042"/>
-      <joint_properties friction="0.0"/>
+      <dynamics friction="0.0"/>
     </joint>
     <link name="${prefix}_thumb_temp_base">
@@ -780,5 +780,5 @@
       <axis xyz="0 0 -1"/>
       <limit effort="0.95" velocity="8.48" lower="-0.349" upper="2.094"/>
-      <joint_properties friction="0.0"/>
+      <dynamics friction="0.0"/>
     </joint>
     <joint name="${prefix}_13" type="revolute">
@@ -788,5 +788,5 @@
       <axis xyz="0 0 -1"/>
       <limit effort="0.95" velocity="8.48" lower="-0.47" upper="2.443"/>
-      <joint_properties friction="0.0"/>
+      <dynamics friction="0.0"/>
     </joint>
     <joint name="${prefix}_14" type="revolute">
@@ -796,5 +796,5 @@
       <axis xyz="0 0 -1"/>
       <limit effort="0.95" velocity="8.48" lower="-1.20" upper="1.90"/>
-      <joint_properties friction="0.0"/>
+      <dynamics friction="0.0"/>
     </joint>
     <joint name="${prefix}_15" type="revolute">
@@ -804,5 +804,5 @@
       <axis xyz="0 0 -1"/>
       <limit effort="0.95" velocity="8.48" lower="-1.34" upper="1.88"/>
-      <joint_properties friction="0.0"/>
+      <dynamics friction="0.0"/>
     </joint>
     <!--  virtual auxiliary link-->
